File: keyboard.kicad_pcb (KiCad board)
At the start: 2 copper layers, 390 x 130 mm, 179 parts, among them SW1 SW_Push, SW10 SW_Push, SW11 SW_Push, SW12 SW_Push, SW13 SW_Push, SW14 SW_Push, SW15 SW_Push, SW16 RotaryEncoder, SW17 SW_Push, SW18 SW_Push, SW19 SW_Push, SW2 SW_Push, SW20 SW_Push, SW21 SW_Push, SW22 SW_Push, SW23 SW_Push, SW24 SW_Push, SW25 SW_Push, SW26 SW_Push, SW27 SW_Push, SW28 SW_Push, SW29 SW_Push, SW3 SW_Push, SW30 SW_Push, SW31 SW_Push, SW32 SW_Push, SW33 SW_Push, SW34 SW_Push, SW35 SW_Push, SW36 SW_Push, SW37 SW_Push, SW38 SW_Push, SW39 SW_Push, SW4 SW_Push, SW40 SW_Push, SW41 SW_Push, SW42 SW_Push, SW43 SW_Push, SW44 SW_Push, SW45 SW_Push, SW46 SW_Push, SW47 SW_Push, SW48 SW_Push, SW49 SW_Push, SW5 SW_Push, SW50 SW_Push, SW51 SW_Push, SW52 SW_Push, SW53 SW_Push, SW54 SW_Push, SW55 SW_Push, SW56 SW_Push, SW57 SW_Push, SW58 SW_Push, SW59 SW_Push, SW6 SW_Push, SW60 SW_Push, SW61 SW_Push, SW62 SW_Push, SW63 SW_Push, SW64 SW_Push, SW65 SW_Push, SW66 SW_Push, SW67 SW_Push, SW68 SW_Push, SW69 SW_Push, SW7 SW_Push, SW70 SW_Push, SW71 SW_Push, SW72 SW_Push, SW73 SW_Push, SW74 SW_Push, SW75 SW_Push, SW76 SW_Push, SW77 SW_Push, SW78 SW_Push, SW79 SW_Push, SW8 SW_Push, SW80 SW_Push, SW81 SW_Push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

Commit message: Arranged keys in layout on pcb
Parts:
- removed D11: 1N4148, PCM_marbastlib-mx:SW_MX_1u
- removed D66, D75, D84: 1N4148, Diode_THT:D_DO-35_SOD27_P7.62mm_Horizontal
- removed S1: MX_stab, PCM_marbastlib-mx:STAB_MX_P_3u
- removed S2, S5, S6: MX_stab, PCM_marbastlib-mx:STAB_MX_P_2u
- removed S8: MX_stab, PCM_marbastlib-mx:STAB_MX_P_4u
- removed SW14, SW31, SW48: SW_Push, PCM_marbastlib-mx:SW_MX_1u
- added D46: 1N4148, Diode_THT:D_DO-35_SOD27_P7.62mm_Horizontal, B.Cu at (49.0, -93.7)
- added ST28: STAB_MX_2u, PCM_marbastlib-mx:STAB_MX_2u, F.Cu at (282.1, -97.8)
- added ST61: STAB_MX_2.25u, PCM_marbastlib-mx:STAB_MX_2.25u, F.Cu at (279.6, -59.5)
- added ST62: STAB_MX_2.25u, PCM_marbastlib-mx:STAB_MX_2.25u, F.Cu at (36.7, -41.1)
- added ST73: STAB_MX_2.75u, PCM_marbastlib-mx:STAB_MX_2.75u, F.Cu at (274.9, -40.3)
- added ST78: STAB_MX_6.25u, PCM_marbastlib-mx:STAB_MX_6.25u, F.Cu at (146.0, -21.0)
- added SW16: SW_Push, PCM_marbastlib-mx:SW_MX_1u, F.Cu at (43.9, -97.7)
- D1, D10, D12, D13, D14, D15, D16, D17, D18, D19, D2, D20, D21, D22, D23, D24, D25, D26, D27, D28, D29, D3, D30, D31, D32, D33, D34, D35, D36, D37, D38, D39, D4, D40, D41, D42, D43, D44, D45, D46, D47, D48, D49, D5, D50, D51, D52, D53, D54, D55, D56, D57, D58, D59, D6, D60, D61, D62, D63, D64, D65, D67, D68, D69, D7, D70, D71, D72, D73, D74, D76, D77, D78, D79, D8, D80, D81, D82, D83, D9: moved to B.Cu
- moved SW10 360.7 mm to (234.3, -126.2)
- moved SW30 344.5 mm to (334.3, -97.6)
- moved SW9 334.1 mm to (205.8, -126.2)
- moved SW29 320.4 mm to (315.3, -97.6)
- moved SW16 317.4 mm to (319.4, -129.5)
- moved D47 314.5 mm to (29.9, -122.2), turned to 90 degrees
- moved SW8 312.3 mm to (186.7, -126.2)
- moved SW44 311.2 mm to (262.9, -78.5)
- moved D18 304.5 mm to (68.0, -122.2), turned to 90 degrees
- moved SW22 298.5 mm to (158.1, -97.6)
- moved SW13 292.3 mm to (291.5, -126.2)
- moved SW7 291.0 mm to (167.7, -126.2)
- moved SW43 288.6 mm to (243.9, -78.5)
- moved D49 287.8 mm to (277.5, -122.2), turned to 90 degrees
- moved D46 287.6 mm to (29.9, -93.6), turned to 90 degrees
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Routing:
- net /Net-(D78-K): track 0.00 -> 20.3 mm
- net /Net-(D58-K): track 0.00 -> 10.1 mm
- net /Net-(D47-K): track 0.00 -> 10.1 mm
- net /Net-(D36-K): track 0.00 -> 10.1 mm
- net /Net-(D3-K): track 0.00 -> 10.1 mm
- net Net-(D65-K): track 0.00 -> 10.1 mm
- net /Net-(D76-K): track 0.00 -> 10.1 mm
- net /Net-(D54-K): track 0.00 -> 10.1 mm
- net /Net-(D24-K): track 0.00 -> 10.1 mm
- net /Net-(D2-K): track 0.00 -> 10.1 mm
- net /Net-(D13-K): track 0.00 -> 10.1 mm
- net /Net-(D9-K): track 0.00 -> 10.1 mm
- net /Net-(D7-K): track 0.00 -> 10.1 mm
- net /Net-(D51-K): track 0.00 -> 10.1 mm
- net /Net-(D31-K): track 0.00 -> 10.1 mm
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Other:
- board size 390 x 130 mm -> 371.5 x 147 mm

Commit message: Partially fixed layout in pcb
Parts:
- removed the D46 at (49.0, -93.7)
- removed the D46 at (29.9, -93.6)
- removed D83: 1N4148, Diode_THT:D_DO-35_SOD27_P7.62mm_Horizontal
- removed the H2 at (214.3, -50.4)
- removed ST28: STAB_MX_2u, PCM_marbastlib-mx:STAB_MX_2u
- removed ST61, ST62: STAB_MX_2.25u, PCM_marbastlib-mx:STAB_MX_2.25u
- removed ST78: STAB_MX_6.25u, PCM_marbastlib-mx:STAB_MX_6.25u
- removed the SW16 at (43.9, -97.7)
- removed the SW16 at (319.4, -129.5)
- removed SW83, SW84, SW85: SW_Push, PCM_marbastlib-mx:SW_MX_1u
- added D11: 1N4148, Diode_THT:D_DO-35_SOD27_P7.62mm_Horizontal, F.Cu at (61.7, -59.5)
- added D46: 1N4148, Diode_THT:D_DO-35_SOD27_P7.62mm_Horizontal, F.Cu at (199.8, -97.6)
- added D66: 1N4148, Diode_THT:D_DO-35_SOD27_P7.62mm_Horizontal, F.Cu at (245.0, -21.4)
- added D75: 1N4148, Diode_THT:D_DO-35_SOD27_P7.62mm_Horizontal, F.Cu at (318.9, -97.6)
- added H3: MountingHole, MountingHole:MountingHole_2.1mm, F.Cu at (130.3, 202.4)
- added ROT1: RotaryEncoder, Rotary_Encoder:RotaryEncoder_Alps_EC11E_Vertical_H20mm, F.Cu at (315.4, -129.5)
- added ST27: MX_stab, PCM_marbastlib-mx:STAB_MX_P_2u, F.Cu at (285.5, -97.6)
- added ST44: MX_stab, PCM_marbastlib-mx:STAB_MX_P_6.25u, F.Cu at (149.8, -21.4)
- added ST58: MX_stab, PCM_marbastlib-mx:STAB_MX_P_2.25u, F.Cu at (283.1, -59.5)
- added ST59: MX_stab, PCM_marbastlib-mx:STAB_MX_P_2.25u, F.Cu at (40.2, -40.5)
- added SW14: SW_Push, PCM_marbastlib-mx:SW_MX_1u, F.Cu at (28.3, -97.6)
- added SW16: SW_Push, PCM_marbastlib-mx:SW_MX_1u, F.Cu at (66.4, -97.6)
- added SW31: SW_Push, PCM_marbastlib-mx:SW_MX_1u, F.Cu at (56.9, -78.5)
- added SW48: SW_Push, PCM_marbastlib-mx:SW_MX_1u, F.Cu at (80.7, -59.5)
- D1, D10, D12, D13, D14, D15, D16, D17, D18, D19, D2, D20, D21, D22, D23, D24, D25, D26, D27, D28, D3, D30, D31, D32, D33, D34, D35, D36, D37, D38, D39, D4, D40, D41, D42, D43, D44, D45, D47, D48, D49, D5, D50, D51, D52, D53, D54, D55, D56, D57, D58, D59, D6, D60, D61, D62, D63, D64, D65, D67, D68, D69, D7, D70, D71, D72, D73, D74, D76, D77, D78, D79, D8, D80, D81, D82, D9: moved to F.Cu
- D29: footprint Diode_THT:D_DO-35_SOD27_P7.62mm_Horizontal -> PCM_marbastlib-mx:SW_MX_1u; moved to F.Cu
- ST73: value STAB_MX_2.75u -> MX_stab; footprint PCM_marbastlib-mx:STAB_MX_2.75u -> PCM_marbastlib-mx:STAB_MX_P_2.75u
- moved SW30 301.8 mm to (33.1, -78.5)
- moved D10 282.5 mm to (56.9, -78.5), turned to 0 degrees
- moved SW46 280.5 mm to (35.5, -59.5)
- moved SW47 273.3 mm to (61.7, -59.5)
- moved D9 266.3 mm to (66.4, -97.6), turned to 0 degrees
- moved D77 257.9 mm to (318.9, -21.4), turned to 0 degrees
- moved SW74 256.7 mm to (78.3, -21.4)
- moved D3 254.4 mm to (33.1, -78.5), turned to 0 degrees
- moved D82 242.8 mm to (357.0, -21.4), turned to 0 degrees
- moved D7 240.4 mm to (47.4, -97.6), turned to 0 degrees
- moved D76 230.9 mm to (318.9, -78.5), turned to 0 degrees
- moved D67 223.6 mm to (295.0, -126.2), turned to 0 degrees
- moved H1 221.6 mm to (9.00, -139.5)
- moved ST73 221.2 mm to (54.5, -21.4)
- moved SW73 221.1 mm to (54.5, -21.4)
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- renumbered H4 to H2, H5 to H4
Connections:
- D10 pad 1: /Net-(D71-K) -> Net-(D10-K)
- D10 pad 2: /ROW4 -> /ROW2
- D12 pad 1: /Net-(D3-K) -> Net-(D12-K)
- D12 pad 2: /ROW0 -> /ROW5
- D13 pad 1: /Net-(D21-K) -> Net-(D13-K)
- D13 pad 2: /ROW1 -> /ROW0
- D14 pad 1: /Net-(D38-K) -> Net-(D14-K)
- D14 pad 2: /ROW2 -> /ROW1
- D15 pad 1: /Net-(D55-K) -> Net-(D15-K)
- D15 pad 2: /ROW3 -> /ROW2
- D16 pad 1: /Net-(D72-K) -> Net-(D16-K)
- D16 pad 2: /ROW4 -> /ROW3
- D17 pad 1: /Net-(D4-K) -> Net-(D17-K)
- D17 pad 2: /ROW0 -> /ROW4
- D18 pad 1: /Net-(D22-K) -> Net-(D18-K)
- D18 pad 2: /ROW1 -> /ROW5
- D19 pad 1: /Net-(D39-K) -> Net-(D19-K)
- D19 pad 2: /ROW2 -> /ROW0
- D2 pad 1: /Net-(D19-K) -> Net-(D2-K)
- D20 pad 1: /Net-(D56-K) -> Net-(D20-K)
- D20 pad 2: /ROW3 -> /ROW1
- D21 pad 1: /Net-(D73-K) -> Net-(D21-K)
- D21 pad 2: /ROW4 -> /ROW2
- D22 pad 1: /Net-(D5-K) -> Net-(D22-K)
- D22 pad 2: /ROW0 -> /ROW3
- D23 pad 2: /ROW1 -> /ROW4
- D24 pad 1: /Net-(D40-K) -> Net-(D24-K)
- D24 pad 2: /ROW2 -> /ROW0
- D25 pad 1: /Net-(D57-K) -> Net-(D25-K)
- D25 pad 2: /ROW3 -> /ROW1
- D26 pad 1: /Net-(D74-K) -> Net-(D26-K)
- D26 pad 2: /ROW4 -> /ROW2
- D27 pad 1: /Net-(D7-K) -> Net-(D27-K)
- D27 pad 2: /ROW0 -> /ROW3
- D28 pad 1: /Net-(D24-K) -> Net-(D28-K)
- D28 pad 2: /ROW1 -> /ROW4
- D29 pad 1: /Net-(D41-K) -> Net-(D29-K)
- D29 pad 2: /ROW2 -> /ROW0
- D3 pad 1: /Net-(D36-K) -> Net-(D3-K)
- D30 pad 1: /Net-(D58-K) -> Net-(D30-K)
- D30 pad 2: /ROW3 -> /ROW1
- D31 pad 1: /Net-(D75-K) -> Net-(D31-K)
- D31 pad 2: /ROW4 -> /ROW2
- D32 pad 1: /Net-(D8-K) -> Net-(D32-K)
- D32 pad 2: /ROW0 -> /ROW3
- D33 pad 1: /Net-(D25-K) -> Net-(D33-K)
- D33 pad 2: /ROW1 -> /ROW4
- D34 pad 1: /Net-(D42-K) -> Net-(D34-K)
- D34 pad 2: /ROW2 -> /ROW0
- D35 pad 1: /Net-(D59-K) -> Net-(D35-K)
- D35 pad 2: /ROW3 -> /ROW1
- D36 pad 1: /Net-(D76-K) -> Net-(D36-K)
- D36 pad 2: /ROW5 -> /ROW2
- D37 pad 1: /Net-(D9-K) -> Net-(D37-K)
- D37 pad 2: /ROW0 -> /ROW3
- D38 pad 1: /Net-(D26-K) -> Net-(D38-K)
- D38 pad 2: /ROW1 -> /ROW4
- D39 pad 1: /Net-(D43-K) -> Net-(D39-K)
- D39 pad 2: /ROW2 -> /ROW0
- D4 pad 1: /Net-(D53-K) -> Net-(D4-K)
- D40 pad 1: /Net-(D60-K) -> Net-(D40-K)
- D40 pad 2: /ROW3 -> /ROW1
- D41 pad 1: /Net-(D77-K) -> Net-(D41-K)
- D41 pad 2: /ROW5 -> /ROW2
- D42 pad 1: /Net-(D10-K) -> Net-(D42-K)
- D42 pad 2: /ROW0 -> /ROW3
- D43 pad 1: /Net-(D27-K) -> Net-(D43-K)
- D43 pad 2: /ROW1 -> /ROW4
- D44 pad 2: /ROW2 -> /ROW5
- D45 pad 1: /Net-(D61-K) -> Net-(D45-K)
- D45 pad 2: /ROW3 -> /ROW0
- D47 pad 1: /Net-(D11-K) -> Net-(D47-K)
- D47 pad 2: /ROW0 -> /ROW2
- D48 pad 1: /Net-(D28-K) -> Net-(D48-K)
- D48 pad 2: /ROW1 -> /ROW3
- D49 pad 1: /Net-(D45-K) -> Net-(D49-K)
- D49 pad 2: /ROW2 -> /ROW4
- D5 pad 1: /Net-(D70-K) -> Net-(D5-K)
- D50 pad 1: /Net-(D62-K) -> Net-(D50-K)
- D50 pad 2: /ROW3 -> /ROW0
- D51 pad 2: /ROW5 -> /ROW1
- D52 pad 1: /Net-(D12-K) -> Net-(D52-K)
- D52 pad 2: /ROW0 -> /ROW2
- D53 pad 1: /Net-(D29-K) -> Net-(D53-K)
- D53 pad 2: /ROW1 -> /ROW3
- D54 pad 1: /Net-(D46-K) -> Net-(D54-K)
- D54 pad 2: /ROW2 -> /ROW4
- D55 pad 1: /Net-(D63-K) -> Net-(D55-K)
- D55 pad 2: /ROW3 -> /ROW0
- D56 pad 1: /Net-(D80-K) -> Net-(D56-K)
- D56 pad 2: /ROW5 -> /ROW1
- D57 pad 1: /Net-(D13-K) -> Net-(D57-K)
- D57 pad 2: /ROW0 -> /ROW2
- D58 pad 1: /Net-(D30-K) -> Net-(D58-K)
- D58 pad 2: /ROW1 -> /ROW3
- D59 pad 1: /Net-(D47-K) -> Net-(D59-K)
- D59 pad 2: /ROW2 -> /ROW4
- D6 pad 1: /Net-(D2-K) -> Net-(D6-K)
- D6 pad 2: /ROW0 -> /ROW5
- D60 pad 1: /Net-(D64-K) -> Net-(D60-K)
- D60 pad 2: /ROW4 -> /ROW5
- D61 pad 1: /Net-(D81-K) -> Net-(D61-K)
- D61 pad 2: /ROW5 -> /ROW0
- D62 pad 2: /ROW0 -> /ROW1
- D63 pad 1: /Net-(D31-K) -> Net-(D63-K)
- D63 pad 2: /ROW1 -> /ROW2
- D64 pad 1: /Net-(D48-K) -> Net-(D64-K)
- D64 pad 2: /ROW2 -> /ROW3
- D67 pad 1: /Net-(D15-K) -> Net-(D67-K)
- D68 pad 1: /Net-(D32-K) -> Net-(D68-K)
- D68 pad 2: /ROW1 -> /ROW2
- D69 pad 1: /Net-(D49-K) -> Net-(D69-K)
- D69 pad 2: /ROW2 -> /ROW5
- D7 pad 1: /Net-(D20-K) -> Net-(D7-K)
- D70 pad 1: /Net-(D66-K) -> Net-(D70-K)
- D70 pad 2: /ROW4 -> /ROW5
- D71 pad 1: /Net-(D83-K) -> Net-(D71-K)
- D71 pad 2: /ROW5 -> /ROW1
- D72 pad 1: /Net-(D16-K) -> Net-(D72-K)
- D72 pad 2: /ROW0 -> /ROW2
- D73 pad 1: /Net-(D33-K) -> Net-(D73-K)
- D73 pad 2: /ROW1 -> /ROW3
- D74 pad 1: /Net-(D50-K) -> Net-(D74-K)
- D74 pad 2: /ROW2 -> /ROW4
- D76 pad 1: /Net-(D84-K) -> Net-(D76-K)
- D76 pad 2: /ROW5 -> /ROW2
- D77 pad 1: /Net-(D17-K) -> Net-(D77-K)
- D77 pad 2: /ROW1 -> /ROW5
- D78 pad 1: /Net-(D34-K) -> Net-(D78-K)
- D78 pad 2: /ROW2 -> /ROW1
- D79 pad 1: /Net-(D51-K) -> Net-(D79-K)
- D79 pad 2: /ROW3 -> /ROW2
- D8 pad 1: /Net-(D37-K) -> Net-(D8-K)
- D8 pad 2: /ROW2 -> /ROW0
- D80 pad 1: /Net-(D68-K) -> Net-(D80-K)
- D81 pad 1: /Net-(D18-K) -> Net-(D81-K)
- D81 pad 2: /ROW1 -> /ROW5
- D82 pad 1: /Net-(D35-K) -> Net-(D82-K)
- D82 pad 2: /ROW2 -> /ROW5
- D9 pad 2: /ROW3 -> /ROW1
- SW1 pad 1: /COL11 -> /COL0
- SW1 pad 2: /Net-(D11-K) -> Net-(D1-K)
- SW10 pad 1: /COL6 -> /COL10
- SW10 pad 2: Net-(D23-K) -> Net-(D50-K)
- SW11 pad 1: /COL0 -> /COL11
- SW11 pad 2: /Net-(D34-K) -> Net-(D55-K)
- SW12 pad 2: /Net-(D45-K) -> Net-(D61-K)
- SW13 pad 1: /COL6 -> /COL13
- SW13 pad 2: /Net-(D56-K) -> Net-(D67-K)
- SW15 pad 1: /COL3 -> /COL1
- SW15 pad 2: /Net-(D78-K) -> Net-(D7-K)
- SW17 pad 1: /COL2 -> /COL3
- SW17 pad 2: /Net-(D2-K) -> Net-(D14-K)
- SW18 pad 1: /COL13 -> /COL4
- SW18 pad 2: /Net-(D13-K) -> Net-(D20-K)
- SW19 pad 1: /COL7 -> /COL5
- SW19 pad 2: /Net-(D24-K) -> Net-(D25-K)
- SW2 pad 1: /COL5 -> /COL2
- SW2 pad 2: /Net-(D22-K) -> Net-(D8-K)
- SW20 pad 1: /COL2 -> /COL6
- SW20 pad 2: /Net-(D35-K) -> Net-(D30-K)
- SW21 pad 1: /COL13 -> /COL7
- SW21 pad 2: /Net-(D46-K) -> Net-(D35-K)
- SW22 pad 1: /COL7 -> /COL8
- SW22 pad 2: /Net-(D57-K) -> Net-(D40-K)
- SW23 pad 1: /COL6 -> /COL9
- SW23 pad 2: /Net-(D68-K) -> Net-(D46-K)
- SW24 pad 1: /COL8 -> /COL10
- SW25 pad 1: /COL3 -> /COL11
- SW25 pad 2: /Net-(D3-K) -> Net-(D56-K)
- SW26 pad 1: /COL15 -> /COL12
- SW27 pad 1: /COL8 -> /COL14
- SW27 pad 2: /Net-(D25-K) -> Net-(D71-K)
- SW28 pad 1: /COL3 -> /COL15
- SW28 pad 2: /Net-(D36-K) -> Net-(D75-K)
- SW29 pad 1: /COL14 -> /COL16
- SW29 pad 2: /Net-(D47-K) -> Net-(D78-K)
- SW3 pad 1: /COL17 -> /COL3
- SW3 pad 2: /Net-(D33-K) -> Net-(D13-K)
- SW30 pad 1: /COL8 -> /COL0
- SW30 pad 2: /Net-(D58-K) -> Net-(D3-K)
- SW32 pad 1: /COL13 -> /COL3
- SW32 pad 2: /Net-(D80-K) -> Net-(D15-K)
- SW33 pad 2: /Net-(D4-K) -> Net-(D21-K)
- SW34 pad 1: /COL16 -> /COL5
- SW34 pad 2: /Net-(D15-K) -> Net-(D26-K)
- SW35 pad 1: /COL9 -> /COL6
- SW35 pad 2: /Net-(D26-K) -> Net-(D31-K)
- SW36 pad 1: /COL4 -> /COL7
- SW36 pad 2: /Net-(D37-K) -> Net-(D36-K)
- SW37 pad 1: /COL15 -> /COL8
- SW37 pad 2: /Net-(D48-K) -> Net-(D41-K)
- SW38 pad 2: /Net-(D59-K) -> Net-(D47-K)
- SW39 pad 1: /COL8 -> /COL10
- SW39 pad 2: /Net-(D70-K) -> Net-(D52-K)
- SW4 pad 1: /COL11 -> /COL4
- SW4 pad 2: Net-(D44-K) -> Net-(D19-K)
- SW40 pad 1: /COL14 -> /COL11
- SW40 pad 2: /Net-(D81-K) -> Net-(D57-K)
- SW41 pad 1: /COL5 -> /COL12
- SW41 pad 2: /Net-(D5-K) -> Net-(D63-K)
- SW42 pad 1: /COL17 -> /COL13
- SW42 pad 2: /Net-(D16-K) -> Net-(D68-K)
- SW43 pad 1: /COL10 -> /COL14
- SW43 pad 2: /Net-(D27-K) -> Net-(D72-K)
- SW44 pad 1: /COL5 -> /COL15
- SW44 pad 2: /Net-(D38-K) -> Net-(D76-K)
- SW45 pad 2: /Net-(D49-K) -> Net-(D79-K)
- SW46 pad 1: /COL10 -> /COL0
- SW46 pad 2: /Net-(D60-K) -> Net-(D4-K)
- SW47 pad 1: /COL9 -> /COL2
- SW47 pad 2: /Net-(D71-K) -> Net-(D11-K)
- SW49 pad 1: /COL6 -> /COL4
- SW49 pad 2: /Net-(D6-K) -> Net-(D22-K)
- SW5 pad 2: /Net-(D55-K) -> Net-(D24-K)
- SW50 pad 1: /COL0 -> /COL5
- SW50 pad 2: /Net-(D17-K) -> Net-(D27-K)
- SW51 pad 1: /COL11 -> /COL6
- SW51 pad 2: /Net-(D28-K) -> Net-(D32-K)
- SW52 pad 1: /COL6 -> /COL7
- SW52 pad 2: /Net-(D39-K) -> Net-(D37-K)
- SW53 pad 1: /COL17 -> /COL8
- SW53 pad 2: /Net-(D50-K) -> Net-(D42-K)
- SW54 pad 1: /COL11 -> /COL9
- SW54 pad 2: /Net-(D61-K) -> Net-(D48-K)
- SW55 pad 2: /Net-(D72-K) -> Net-(D53-K)
- SW56 pad 1: /COL16 -> /COL11
- SW56 pad 2: /Net-(D83-K) -> Net-(D58-K)
- SW57 pad 1: /COL7 -> /COL12
- SW57 pad 2: /Net-(D7-K) -> Net-(D64-K)
- SW58 pad 1: /COL1 -> /COL14
- SW58 pad 2: /Net-(D18-K) -> Net-(D73-K)
- SW59 pad 1: /COL12 -> /COL0
- SW59 pad 2: /Net-(D29-K) -> Net-(D5-K)
- SW6 pad 1: /COL4 -> /COL6
- SW6 pad 2: /Net-(D66-K) -> Net-(D29-K)
- SW60 pad 1: /COL7 -> /COL3
- SW60 pad 2: /Net-(D40-K) -> Net-(D17-K)
- SW61 pad 1: /COL0 -> /COL4
- SW61 pad 2: /Net-(D51-K) -> Net-(D23-K)
- SW62 pad 1: /COL12 -> /COL5
- SW62 pad 2: /Net-(D62-K) -> Net-(D28-K)
- SW63 pad 1: /COL11 -> /COL6
- SW63 pad 2: /Net-(D73-K) -> Net-(D33-K)
- SW64 pad 1: /COL17 -> /COL7
- SW64 pad 2: /Net-(D84-K) -> Net-(D38-K)
- SW65 pad 2: /Net-(D8-K) -> Net-(D43-K)
- SW66 pad 1: /COL2 -> /COL9
- SW66 pad 2: /Net-(D19-K) -> Net-(D49-K)
- SW67 pad 1: /COL14 -> /COL10
- SW67 pad 2: /Net-(D30-K) -> Net-(D54-K)
- SW68 pad 1: /COL8 -> /COL11
- SW68 pad 2: /Net-(D41-K) -> Net-(D59-K)
- SW69 pad 1: /COL2 -> /COL12
- SW69 pad 2: /Net-(D52-K) -> Net-(D65-K)
- SW7 pad 1: /COL1 -> /COL7
- SW7 pad 2: /Net-(D77-K) -> Net-(D34-K)
- SW70 pad 2: /Net-(D63-K) -> Net-(D74-K)
- SW71 pad 1: /COL12 -> /COL16
- SW71 pad 2: /Net-(D74-K) -> Net-(D80-K)
- SW72 pad 1: /COL9 -> /COL0
- SW72 pad 2: /Net-(D9-K) -> Net-(D6-K)
- SW73 pad 1: /COL3 -> /COL2
- SW73 pad 2: /Net-(D20-K) -> Net-(D12-K)
- SW74 pad 1: /COL15 -> /COL3
- SW74 pad 2: /Net-(D31-K) -> Net-(D18-K)
- SW75 pad 1: /COL9 -> /COL7
- SW75 pad 2: /Net-(D42-K) -> Net-(D44-K)
- SW76 pad 1: /COL3 -> /COL11
- SW76 pad 2: /Net-(D53-K) -> Net-(D60-K)
- SW77 pad 1: /COL0 -> /COL12
- SW77 pad 2: /Net-(D64-K) -> Net-(D66-K)
- SW78 pad 1: /COL14 -> /COL13
- SW78 pad 2: /Net-(D75-K) -> Net-(D69-K)
- SW79 pad 1: /COL10 -> /COL14
- SW79 pad 2: /Net-(D10-K) -> Net-(D70-K)
- SW8 pad 1: /COL0 -> /COL8
- SW8 pad 2: Net-(D1-K) -> Net-(D39-K)
- SW80 pad 1: /COL4 -> /COL15
- SW80 pad 2: /Net-(D21-K) -> Net-(D77-K)
- SW81 pad 2: /Net-(D32-K) -> Net-(D81-K)
- SW82 pad 1: /COL10 -> /COL17
- SW82 pad 2: /Net-(D43-K) -> Net-(D82-K)
- SW9 pad 1: /COL12 -> /COL9
- SW9 pad 2: /Net-(D12-K) -> Net-(D45-K)
Routing:
- net /Net-(D78-K): track 20.3 -> 0.00 mm
- net /Net-(D58-K): track 10.1 -> 0.00 mm
- net /Net-(D47-K): track 10.1 -> 0.00 mm
- net /Net-(D36-K): track 10.1 -> 0.00 mm
- net /Net-(D3-K): track 10.1 -> 0.00 mm
- net Net-(D9-K): track 10.1 -> 0.00 mm
- net Net-(D65-K): track 10.1 -> 0.00 mm
- net /Net-(D76-K): track 10.1 -> 0.00 mm
- net /Net-(D24-K): track 10.1 -> 0.00 mm
- net /Net-(D2-K): track 10.1 -> 0.00 mm
- net /Net-(D13-K): track 10.1 -> 0.00 mm
- net /Net-(D9-K): track 10.1 -> 0.00 mm
- net /Net-(D7-K): track 10.1 -> 0.00 mm
- net /Net-(D51-K): track 10.1 -> 0.00 mm
- net /Net-(D31-K): track 10.1 -> 0.00 mm
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
Commit message: Added traces in schematic, not completely implemented on pcb
Parts:
- D6: renamed from D29; footprint PCM_marbastlib-mx:SW_MX_1u -> Diode_THT:D_DO-35_SOD27_P7.62mm_Horizontal
- moved H3 425.9 mm to (385.5, -138.5)
- moved A1 90.6 mm to (358.6, -152.3)
- moved H4 19.0 mm to (386.0, -6.50)
- moved H1 6.95 mm to (5.50, -145.5)
- moved H2 3.16 mm to (6.50, -7.00)
- moved D10 2.97 mm to (235.3, -127.6)
- moved D12 2.97 mm to (273.4, -127.6)
- moved D13 2.97 mm to (292.4, -127.6)
- moved D20 2.97 mm to (140.0, -99.0)
- moved D25 2.97 mm to (235.3, -99.0)
- moved D28 2.97 mm to (316.3, -99.0)
- moved D38 2.97 mm to (187.7, -80.0)
- moved D44 2.97 mm to (316.3, -80.0)
- moved D55 2.97 mm to (211.5, -61.0)
- moved D58 2.97 mm to (280.5, -61.0)
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- renumbered D50 to D10, D55 to D11, D61 to D12, D67 to D13, D2 to D14, D7 to D15, D9 to D16, D14 to D17, D20 to D18, D25 to D19, D8 to D2, D30 to D20, D35 to D21, D40 to D22, D46 to D23, D51 to D24, D56 to D25, D62 to D26, D71 to D27, D75 to D28, D78 to D29, D13 to D3, D3 to D30, D10 to D31, D15 to D32, D21 to D33, D26 to D34, D31 to D35, D41 to D37, D47 to D38, D52 to D39, D19 to D4, D57 to D40, D63 to D41, D68 to D42, D72 to D43, D76 to D44, D79 to D45, D4 to D46, D11 to D47, D16 to D48, D22 to D49, D24 to D5, D27 to D50, D32 to D51, D37 to D52, D42 to D53, D48 to D54, D53 to D55, D58 to D56, D64 to D57, D73 to D58, D5 to D59, D17 to D60, D23 to D61, D28 to D62, D33 to D63, D38 to D64, D43 to D65, D49 to D66, D54 to D67, D59 to D68, D65 to D69, D34 to D7, D74 to D70, D80 to D71, D6 to D72, D12 to D73, D18 to D74, D44 to D75, D60 to D76, D66 to D77, D69 to D78, D70 to D79, D39 to D8, D77 to D80, D45 to D9
Connections:
- A1 pad 10: unconnected-(A1-GPIO7-Pad10) -> /COL4
- A1 pad 11: unconnected-(A1-GPIO8-Pad11) -> /COL5
- A1 pad 12: unconnected-(A1-GPIO9-Pad12) -> /COL6
- A1 pad 14: unconnected-(A1-GPIO10-Pad14) -> /COL7
- A1 pad 15: unconnected-(A1-GPIO11-Pad15) -> /COL8
- A1 pad 16: unconnected-(A1-GPIO12-Pad16) -> /COL9
- A1 pad 17: unconnected-(A1-GPIO13-Pad17) -> /COL10
- A1 pad 19: unconnected-(A1-GPIO14-Pad19) -> /COL11
- A1 pad 20: unconnected-(A1-GPIO15-Pad20) -> /COL12
- A1 pad 21: unconnected-(A1-GPIO16-Pad21) -> /COL13
- A1 pad 22: unconnected-(A1-GPIO17-Pad22) -> /COL14
- A1 pad 24: unconnected-(A1-GPIO18-Pad24) -> /COL15
- A1 pad 26: unconnected-(A1-GPIO20-Pad26) -> /COL16
- A1 pad 27: unconnected-(A1-GPIO21-Pad27) -> /COL17
- A1 pad 5: unconnected-(A1-GPIO3-Pad5) -> /COL0
- A1 pad 6: unconnected-(A1-GPIO4-Pad6) -> /COL1
- A1 pad 7: unconnected-(A1-GPIO5-Pad7) -> /COL2
- A1 pad 9: unconnected-(A1-GPIO6-Pad9) -> /COL3
- D34 pad 2: /ROW2 -> unconnected-(D34-A-Pad2)
- D6 pad 2: /ROW0 -> unconnected-(D6-A-Pad2)
- ROT1 pad A: /COL15 -> unconnected-(ROT1-PadA)
- ROT1 pad B: /COL15 -> unconnected-(ROT1-PadB)
- ROT1 pad C: /COL15 -> unconnected-(ROT1-PadC)
Routing:
- net /COL14: track 0.00 -> 131.9 mm
- net /COL0: track 0.00 -> 131.0 mm
- net /COL7: track 0.00 -> 128.9 mm
- net /COL3: track 0.00 -> 127.5 mm
- net /COL2: track 0.00 -> 124.0 mm
- net /COL12: track 0.00 -> 123.5 mm
- net /COL11: track 0.00 -> 123.5 mm
- net /COL13: track 0.00 -> 117.6 mm
- net /COL6: track 0.00 -> 108.7 mm
- net /COL8: track 0.00 -> 107.4 mm
- net /COL10: track 0.00 -> 105.4 mm
- net /COL4: track 0.00 -> 105.0 mm
- net /COL5: track 0.00 -> 104.6 mm
- net /COL9: track 0.00 -> 101.0 mm
- net /COL16: track 0.00 -> 84.8 mm
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Other:
- board size 371.5 x 147 mm -> 395 x 155 mm
